Commit message: URDF: added laser to the new tilt GENERAL: removed ptu_d46_driver dependency from Cmake files and packages

File: fsr_husky_description/urdf/fsr_husky.urdf.xacro (robot description, xacro)
@@ -46,5 +46,5 @@
     <xacro:include filename="$(find fsr_husky_description)/urdf/husky_parts/parts.urdf.xacro" />
     <xacro:include filename="$(find fsr_husky_description)/urdf/fsr_husky_parts/husky_bridge.urdf.xacro" />
-    <!--<xacro:include filename="$(find fsr_husky_description)/urdf/fsr_husky_parts/sick_lms100.urdf.xacro" /> -->
+    <xacro:include filename="$(find fsr_husky_description)/urdf/fsr_husky_parts/sick_lms100.urdf.xacro" />
     <xacro:include filename="$(find fsr_husky_description)/urdf/fsr_husky_parts/alfa_tube2h.urdf.xacro" />
     <xacro:include filename="$(find fsr_husky_description)/urdf/fsr_husky_parts/pointgrey_flea3.urdf.xacro" />
@@ -189,7 +189,7 @@
     <!-- PTU-D46 macro -->
     <!--<ptu_d46 parent="front_husky_bridge" x="0" y="-0.025" z="0.04" rx="0" ry="0" rz="1.5708" />-->
-    <ptu_d46 parent="front_husky_bridge" x="0" y="0.0" z="-0.004" rx="0" ry="0" rz="-1.5708" />
+    <ptu_d46 parent="front_husky_bridge" x="0.05" y="0.0" z="-0.004" rx="0" ry="0" rz="-1.5708" />
     <!-- SICK macro -->
-    <sick_lms100 parent="ptu_d46_tilt_link" x="0.0" y="0.13" z="0.11" rx="0.0" ry="-0.541053905" rz="-1.5708" />
+    <sick_lms100 parent="ptu_d46_tilt_link" x="0.01242" y="0.0" z="0.06360" rx="0.0" ry="0" rz="0" />
     <!-- GPS macro -->
     <gps_antenna parent="back_husky_bridge" x="0" y="0.17" z="0.0" rx="0" ry="0" rz="0" />

File: fsr_husky_description/urdf/fsr_husky_mine_detection.urdf.xacro (robot description, xacro)
@@ -46,5 +46,5 @@
     <xacro:include filename="$(find fsr_husky_description)/urdf/husky_parts/parts.urdf.xacro" />
     <xacro:include filename="$(find fsr_husky_description)/urdf/fsr_husky_parts/husky_bridge.urdf.xacro" />
-    <!--<xacro:include filename="$(find fsr_husky_description)/urdf/fsr_husky_parts/sick_lms100.urdf.xacro" />-->
+    <xacro:include filename="$(find fsr_husky_description)/urdf/fsr_husky_parts/sick_lms100.urdf.xacro" />
     <xacro:include filename="$(find fsr_husky_description)/urdf/fsr_husky_parts/alfa_tube2h.urdf.xacro" />
     <xacro:include filename="$(find fsr_husky_description)/urdf/fsr_husky_parts/pointgrey_flea3.urdf.xacro" />
@@ -190,7 +190,7 @@
     <!-- PTU-D46 macro -->
     <!--<ptu_d46 parent="front_husky_bridge" x="0" y="-0.025" z="0.04" rx="0" ry="0" rz="1.5708" />-->
-    <ptu_d46 parent="front_husky_bridge" x="0" y="0.0" z="-0.004" rx="0" ry="0" rz="-1.5708" />
+    <ptu_d46 parent="front_husky_bridge" x="0.05" y="0.0" z="-0.004" rx="0" ry="0" rz="-1.5708" />
     <!-- SICK macro -->
-    <sick_lms100 parent="ptu_d46_tilt_link" x="0.0" y="0.13" z="0.11" rx="0.0" ry="-0.541053905" rz="-1.5708" />
+    <sick_lms100 parent="ptu_d46_tilt_link" x="0.01242" y="0.0" z="0.06360" rx="0.0" ry="0" rz="0" />
     <!-- GPS macro -->
     <gps_antenna parent="back_husky_bridge" x="0" y="0.17" z="0.0" rx="0" ry="0" rz="0" />

File: fsr_husky_description/urdf/fsr_husky_parts/tilt.urdf.xacro (robot description, xacro)
@@ -105,16 +105,6 @@
 			<dynamics damping="0.008" friction="0.6" />
   		</joint>
+		-->
 		<link name="ptu_d46_tilt_link">
-    			<inertial>
-      				<origin xyz="4.5103E-17 0.019688 0" rpy="0 0 0" />
-      				<mass value="0.036018" />
-      				<inertia
-        				ixx="1.0844E-05"
-        				ixy="-7.4115E-22"
-        				ixz="8.6821E-21"
-        				iyy="2.2806E-05"
-        				iyz="-2.5411E-21"
-        				izz="2.9855E-05" />
-    			</inertial>
     			<visual>
       				<origin xyz="0 0 0" rpy="0 0 0" />
@@ -136,19 +126,11 @@
     		</gazebo>
 		<joint name="ptu_d46_tilt_joint" type="revolute">
-    			<origin xyz="0 0 0.0455" rpy="1.3 0 0" />
-    			<parent link="ptu_d46_pan_link" />
+    			<origin xyz="0 0 0.17274" rpy="0 0 1.57" />
+    			<parent link="ptu_d46_base_link" />
     			<child link="ptu_d46_tilt_link" />
-    			<axis xyz="-1 0 0" />
-    			<limit effort="6.0" lower="-0.5" upper="0.5" velocity="0.5" />
+    			<axis xyz="0 1 0" />
+    			<limit effort="6.0" lower="-1.5" upper="1.5" velocity="1.17" />
 			<dynamics damping="0.008" friction="0.6" />
   		</joint>
-		<transmission name="pan">
-		  <type>transmission_interface/SimpleTransmission</type>
-		  <joint name="ptu_d46_pan_joint"/>
-		  <actuator name="pan_motor">
-		    <hardwareInterface>EffortJointInterface</hardwareInterface>
-		    <mechanicalReduction>1</mechanicalReduction>
-		  </actuator>
-		</transmission>
 		<transmission name="tilt">
 		  <type>transmission_interface/SimpleTransmission</type>
@@ -158,5 +140,5 @@
 		    <mechanicalReduction>1</mechanicalReduction>
 		  </actuator>
-		</transmission> -->
+		</transmission>
 		<!--<gazebo>
 		  <plugin name="gazebo_ros_control" filename="libgazebo_ros_control.so">
