Commit message: URDF: removed model for tilt_link

File: fsr_husky_description/urdf/fsr_husky_parts/tilt.urdf.xacro (robot description, xacro)
@@ -107,5 +107,5 @@
 		-->
 		<link name="ptu_d46_tilt_link">
-    			<visual>
+    			<!--<visual>
       				<origin xyz="0 0 0" rpy="0 0 0" />
       				<geometry>
@@ -119,10 +119,6 @@
 					<mesh filename="package://fsr_husky_description/models/fsr_husky_parts/ptu_d46_tilt_link.stl" />
       				</geometry>
-    			</collision>
+		  </collision> -->
   		</link>
-		<gazebo reference="ptu_d46_tilt_link">
-        		<material>Gazebo/FlatBlack</material>
-        		<turnGravityOff>false</turnGravityOff>
-    		</gazebo>
 		<joint name="ptu_d46_tilt_joint" type="revolute">
     			<origin xyz="0 0 0.17274" rpy="0 0 1.57" />

Commit message: URDF: fix : negative y axis GENERAL: fix: tilt test launchfile fixed

File: fsr_husky_description/urdf/fsr_husky_parts/tilt.urdf.xacro (robot description, xacro)
@@ -125,5 +125,5 @@
     			<parent link="ptu_d46_base_link" />
     			<child link="ptu_d46_tilt_link" />
-    			<axis xyz="0 1 0" />
+    			<axis xyz="0 -1 0" />
     			<limit effort="6.0" lower="-1.5" upper="1.5" velocity="1.17" />
 			<dynamics damping="0.008" friction="0.6" />
