Commit message: Initial commit of the movit package.

File: fsr_husky_description/urdf/arm/fsr_husky_arm.urdf.xacro (robot description, xacro)
@@ -230,4 +230,7 @@
     name="metal_detector_arm_joint"
     type="revolute">
+    <mimic
+      joint="upper_arm_joint"
+      multiplier="-1" />
     <origin
       xyz="0 0 0.8475"
@@ -341,4 +344,6 @@
     name="lower_arm_joint"
     type="revolute">
+    <mimic
+      joint="upper_arm_joint" />
     <origin
       xyz="0 0.0809 -0.011058"

Commit message: Initial commit of the fsr_husky_gazebo package.

File: fsr_husky_description/urdf/arm/fsr_husky_arm.urdf.xacro (robot description, xacro)
@@ -24,5 +24,8 @@
 SOFTWARE, EVEN IF ADVISED OF THE POSSIBILITY OF SUCH DAMAGE.
 -->
-<robot xmlns:xacro="http://ros.org/wiki/xacro" name="fsr_husky_arm">
+<robot xmlns:sensor="http://playerstage.sourceforge.net/gazebo/xmlschema/#sensor"
+	xmlns:controller="http://playerstage.sourceforge.net/gazebo/xmlschema/#controller"
+	xmlns:interface="http://playerstage.sourceforge.net/gazebo/xmlschema/#interface"
+	xmlns:xacro="http://ros.org/wiki/xacro" name="fsr_husky_arm">
 <xacro:macro name="fsr_husky_arm" params="parent x y z rx ry rz">
   <link
@@ -66,4 +69,8 @@
     </collision>
   </link>
+  <gazebo reference="base_arm_link">
+        <material>Gazebo/Grey</material>
+        <turnGravityOff>true</turnGravityOff>
+    </gazebo>
   <joint name="arm_joint" type="fixed">
 			<parent link="${parent}"/>
@@ -111,4 +118,8 @@
     </collision>
   </link>
+  <gazebo reference="arm_axel">
+        <material>Gazebo/Grey</material>
+        <turnGravityOff>true</turnGravityOff>
+    </gazebo>
   <joint
     name="arm_axel_joint"
@@ -169,4 +180,8 @@
     </collision>
   </link>
+  <gazebo reference="upper_arm">
+        <material>Gazebo/Grey</material>
+        <turnGravityOff>true</turnGravityOff>
+    </gazebo>
   <joint
     name="upper_arm_joint"
@@ -227,4 +242,8 @@
     </collision>
   </link>
+  <gazebo reference="metal_detector_arm">
+        <material>Gazebo/Grey</material>
+        <turnGravityOff>true</turnGravityOff>
+    </gazebo>
   <joint
     name="metal_detector_arm_joint"
@@ -288,4 +307,8 @@
     </collision>
   </link>
+  <gazebo reference="metal_detector_antenna">
+        <material>Gazebo/Green</material>
+        <turnGravityOff>true</turnGravityOff>
+    </gazebo>
   <joint
     name="metal_detector_antenna_joint"
@@ -341,4 +364,8 @@
     </collision>
   </link>
+  <gazebo reference="lower_arm">
+        <material>Gazebo/Grey</material>
+        <turnGravityOff>true</turnGravityOff>
+    </gazebo>
   <joint
     name="lower_arm_joint"

File: fsr_husky_description/urdf/fsr_husky_mine_detection.urdf.xacro (robot description, xacro)
@@ -133,7 +133,59 @@
     <husky_wheel fb="front" lr="left" parent="base_link" translateX="1" translateY="1" flipY="-1"/>
     <husky_wheel fb="front" lr="right" parent="base_link" translateX="1" translateY="-1" flipY="-1"/>
+    <!-- DECORATIONS -->
+   <!-- Top Plate -->
+    <husky_part parent="base_footprint" name="top_plate" mesh="top_plate"
+          colour="Yellow"
+          translateX="0.0" translateY="0.0" translateZ="${wheel_x_size/2 - base_z_origin_to_wheel_origin}"
+          rotateX="0.0" rotateY="0.0" rotateZ="0.0"/>
+    <gazebo reference="base_footprint_top_plate_part">
+        <material>Gazebo/Yellow</material>
+	<turnGravityOff>false</turnGravityOff>
+    </gazebo>
+    <!-- User Rail -->
+    <husky_part parent="base_footprint" name="user_rail" mesh="user_rail"
+          colour="DarkGray"
+          translateX="0.272" translateY="0.0" translateZ="${0.245 + wheel_x_size/2 - base_z_origin_to_wheel_origin}"
+          rotateX="0.0" rotateY="0.0" rotateZ="0.0"/>
+    <gazebo reference="base_footprint_user_rail_part">
+        <material>Gazebo/Grey</material>
+	<turnGravityOff>false</turnGravityOff>
+    </gazebo>
+    <!-- Bumpers -->
+    <husky_part parent="base_footprint" name="front_bumper" mesh="bumper"
+          colour="DarkGray"
+          translateX="0.490" translateY="0.0" translateZ="${0.091 + wheel_x_size/2 - base_z_origin_to_wheel_origin}"
+          rotateX="0.0" rotateY="0.0" rotateZ="0.0"/>
+    <gazebo reference="base_footprint_front_bumper_part">
+        <material>Gazebo/FlatBlack</material>
+	<turnGravityOff>false</turnGravityOff>
+    </gazebo>
+    <husky_part parent="base_footprint" name="rear_bumper" mesh="bumper"
+          colour="DarkGray"
+          translateX="-0.48" translateY="0.0" translateZ="${0.091 + wheel_x_size/2 - base_z_origin_to_wheel_origin}"
+          rotateX="0.0" rotateY="0.0" rotateZ="3.14"/>
+    <gazebo reference="base_footprint_rear_bumper_part">
+        <material>Gazebo/FlatBlack</material>
+	<turnGravityOff>false</turnGravityOff>
+    </gazebo>
+    <gazebo>
+	<plugin name="husky_diff_controller" filename="libhusky_gazebo_plugins.so">
+	    <alwaysOn>true</alwaysOn>
+            <updateRate>100.0</updateRate>
+            <backLeftJoint>joint_back_left_wheel</backLeftJoint>
+            <backRightJoint>joint_back_right_wheel</backRightJoint>
+            <frontLeftJoint>joint_front_left_wheel</frontLeftJoint>
+            <frontRightJoint>joint_front_right_wheel</frontRightJoint>
+            <wheelSeparation>${base_y_size}</wheelSeparation>
+            <wheelDiameter>${wheel_x_size}</wheelDiameter>
+            <torque>35</torque>
+        </plugin>
+    </gazebo>
+    <!-- FSR Husky Stuff -->
     <!-- BRIDGE macros -->
     <husky_bridge prefix="front" parent="base_link" x="0.17" y="0" z="${base_z_size}" rx="0" ry="0" rz="0" />
     <husky_bridge prefix="back" parent="base_link" x="-0.18" y="0" z="${base_z_size}" rx="0" ry="0" rz="0" />
+    <!-- MTi macro -->
+    <mti parent="back_husky_bridge" x="0" y="0" z="0.0" rx="0" ry="0" rz="0" />
     <!-- CAMERA macros -->
     <pointgrey_flea3 prefix="left" parent="front_husky_bridge" base_offset="-0.13" camera_offset="-0.05" camera_r="0" camera_p="0" camera_y="0" />
@@ -145,52 +197,7 @@
     <!-- GPS macro -->
     <gps_antenna parent="back_husky_bridge" x="0" y="0.17" z="0.0" rx="0" ry="0" rz="0" />
+    <!-- WiFi Antenna -->
+    <alfa_tube2h parent="back_husky_bridge" x="0" y="-0.17" z="0" rx="0" ry="0" rz="0" />
     <!-- FSR Husky De-mining Arm -->
     <fsr_husky_arm parent="base_link" x="0.120" y="-0.15" z="${base_z_size}" rx="0" ry="0" rz="0" />
-    <!-- DECORATIONS -->
-    <!-- WiFi Antenna -->
-    <alfa_tube2h parent="back_husky_bridge" x="0" y="-0.17" z="0" rx="0" ry="0" rz="0" />
-   <!-- Top Plate -->
-    <husky_part parent="base_footprint" name="top_plate" mesh="top_plate"
-          colour="Yellow"
-          translateX="0.0" translateY="0.0" translateZ="${wheel_x_size/2 - base_z_origin_to_wheel_origin}"
-          rotateX="0.0" rotateY="0.0" rotateZ="0.0"/>
-    <gazebo reference="base_footprint_top_plate_part">
-        <material>Gazebo/Yellow</material>
-    </gazebo>
-    <!-- User Rail -->
-    <husky_part parent="base_footprint" name="user_rail" mesh="user_rail"
-          colour="DarkGray"
-          translateX="0.272" translateY="0.0" translateZ="${0.245 + wheel_x_size/2 - base_z_origin_to_wheel_origin}"
-          rotateX="0.0" rotateY="0.0" rotateZ="0.0"/>
-    <gazebo reference="base_footprint_user_rail_part">
-        <material>Gazebo/Grey</material>
-    </gazebo>
-    <!-- Bumpers -->
-    <husky_part parent="base_footprint" name="front_bumper" mesh="bumper"
-          colour="DarkGray"
-          translateX="0.490" translateY="0.0" translateZ="${0.091 + wheel_x_size/2 - base_z_origin_to_wheel_origin}"
-          rotateX="0.0" rotateY="0.0" rotateZ="0.0"/>
-    <gazebo reference="base_footprint_front_bumper_part">
-        <material>Gazebo/FlatBlack</material>
-    </gazebo>
-    <husky_part parent="base_footprint" name="rear_bumper" mesh="bumper"
-          colour="DarkGray"
-          translateX="-0.48" translateY="0.0" translateZ="${0.091 + wheel_x_size/2 - base_z_origin_to_wheel_origin}"
-          rotateX="0.0" rotateY="0.0" rotateZ="3.14"/>
-    <gazebo reference="base_footprint_rear_bumper_part">
-        <material>Gazebo/FlatBlack</material>
-    </gazebo>
-    <gazebo>
-	    <plugin name="husky_diff_controller" filename="libhusky_gazebo_plugins.so">
-		    <alwaysOn>true</alwaysOn>
-            <updateRate>100.0</updateRate>
-            <backLeftJoint>joint_back_left_wheel</backLeftJoint>
-            <backRightJoint>joint_back_right_wheel</backRightJoint>
-            <frontLeftJoint>joint_front_left_wheel</frontLeftJoint>
-            <frontRightJoint>joint_front_right_wheel</frontRightJoint>
-            <wheelSeparation>${base_y_size}</wheelSeparation>
-            <wheelDiameter>${wheel_x_size}</wheelDiameter>
-            <torque>35</torque>
-        </plugin>
-    </gazebo>
 </robot>

File: fsr_husky_description/urdf/parts/alfa_tube2h.urdf.xacro (robot description, xacro)
@@ -52,4 +52,8 @@
     			</collision>
   		</link>
+		<gazebo reference="alfa_tube2h">
+        		<material>Gazebo/White</material>
+        		<turnGravityOff>false</turnGravityOff>
+    		</gazebo>
 		<joint name="joint_alfa_tub2h" type="fixed">
 			<parent link="${parent}"/>
@@ -72,4 +76,8 @@
     			</collision>
   		</link>
+		<gazebo reference="wifi_antenna">
+        		<material>Gazebo/White</material>
+        		<turnGravityOff>false</turnGravityOff>
+    		</gazebo>
 		<joint name="joint_wifi_anetnna" type="fixed">
 			<parent link="alfa_tube2h"/>

File: fsr_husky_description/urdf/parts/gps_antenna.urdf.xacro (robot description, xacro)
@@ -63,4 +63,8 @@
     			</collision>
   		</link>
+		<gazebo reference="gps_antenna">
+        		<material>Gazebo/White</material>
+        		<turnGravityOff>false</turnGravityOff>
+    		</gazebo>
 		<joint name="gps_anetnna_joint" type="fixed">
 			<parent link="${parent}"/>

File: fsr_husky_description/urdf/parts/husky_bridge.urdf.xacro (robot description, xacro)
@@ -57,4 +57,8 @@
     			</collision>
 		</link>
+		<gazebo reference="${prefix}_husky_bridge">
+	        	<material>Gazebo/Grey</material>
+	        	<turnGravityOff>false</turnGravityOff>
+    		</gazebo>
 		<joint name="joint_${prefix}_husky_bridge" type="fixed">
 			<parent link="${parent}"/>

File: fsr_husky_description/urdf/parts/mti.urdf.xacro (robot description, xacro)
@@ -55,4 +55,8 @@
 			<origin xyz="${x} ${y} ${z+mti_height/2}" rpy="${rx} ${ry} ${rz}" />
 		</joint>
+		<gazebo reference="mti">
+        		<material>Gazebo/Orange</material>
+        		<turnGravityOff>false</turnGravityOff>
+    		</gazebo>
 	</xacro:macro>
 </robot>

File: fsr_husky_description/urdf/parts/pointgrey_flea3.urdf.xacro (robot description, xacro)
@@ -55,4 +55,8 @@
     			</collision>
   		</link>
+		<gazebo reference="${prefix}_camera_base">
+        		<material>Gazebo/Grey</material>
+       			 <turnGravityOff>false</turnGravityOff>
+    		</gazebo>
 		<joint name="joint_${prefix}_camera_base" type="fixed">
 			<parent link="${parent}"/>
@@ -76,4 +80,8 @@
     			</collision>
   		</link>
+		<gazebo reference="${prefix}_camera_standoff">
+        		<material>Gazebo/Grey</material>
+       			 <turnGravityOff>false</turnGravityOff>
+    		</gazebo>
 		<joint name="joint_${prefix}_camera_standoff" type="fixed">
 			<parent link="${prefix}_camera_base"/>
@@ -97,4 +105,8 @@
     			</collision>
   		</link>
+		<gazebo reference="${prefix}_camera">
+        		<material>Gazebo/Black</material>
+       			 <turnGravityOff>false</turnGravityOff>
+    		</gazebo>
 		<joint name="joint_${prefix}_camera" type="fixed">
 			<parent link="${prefix}_camera_standoff"/>
@@ -123,4 +135,45 @@
 			<origin xyz="0 0 ${flea_size/2+lense_length/2}" rpy="${camera_r} ${camera_p} ${camera_y}" />
 		</joint>
+		<!-- camera -->
+  		<gazebo reference="${prefix}_lense">
+			<material>Gazebo/Black</material>
+       			 <turnGravityOff>false</turnGravityOff>
+    			<sensor type="camera" name="${prefix}_camera">
+      				<update_rate>30.0</update_rate>
+      				<camera name="${prefix}_pgr">
+        				<horizontal_fov>1.3962634</horizontal_fov>
+        				<image>
+          					<width>800</width>
+          					<height>800</height>
+          					<format>R8G8B8</format>
+        				</image>
+        				<clip>
+          					<near>0.02</near>
+          					<far>300</far>
+        				</clip>
+        				<noise>
+          					<type>gaussian</type>
+          					<!-- Noise is sampled independently per pixel on each frame.
+               					That pixel's noise value is added to each of its color channels, which at that point lie in the range [0,1]. -->
+          					<mean>0.0</mean>
+          					<stddev>0.007</stddev>
+        				</noise>
+      				</camera>
+      				<plugin name="camera_controller" filename="libgazebo_ros_camera.so">
+        				<alwaysOn>true</alwaysOn>
+        				<updateRate>0.0</updateRate>
+        				<cameraName>${prefix}_camera</cameraName>
+       					<imageTopicName>image_raw</imageTopicName>
+        				<cameraInfoTopicName>camera_info</cameraInfoTopicName>
+        				<frameName>camera_link</frameName>
+        				<hackBaseline>0.07</hackBaseline>
+        				<distortionK1>0.0</distortionK1>
+        				<distortionK2>0.0</distortionK2>
+        				<distortionK3>0.0</distortionK3>
+        				<distortionT1>0.0</distortionT1>
+        				<distortionT2>0.0</distortionT2>
+      				</plugin>
+    			</sensor>
+  		</gazebo>
 	</xacro:macro>
 </robot>

File: fsr_husky_description/urdf/parts/ptu_d46.urdf.xacro (robot description, xacro)
@@ -56,4 +56,8 @@
     			</collision>
   		</link>
+		<gazebo reference="ptu_d46_base_link">
+        		<material>Gazebo/FlatBlack</material>
+        		<turnGravityOff>false</turnGravityOff>
+    		</gazebo>
 		<joint name="ptu_d46_joint" type="fixed">
 			<parent link="${parent}"/>
@@ -87,4 +91,8 @@
     			</collision>
   		</link>
+		<gazebo reference="ptu_d46_pan_link">
+        		<material>Gazebo/FlatBlack</material>
+        		<turnGravityOff>false</turnGravityOff>
+    		</gazebo>
 		<joint name="ptu_d46_pan_joint" type="revolute">
     			<origin xyz="0.026 -0.0215 0.044" rpy="-6.123E-17 0 0" />
@@ -120,4 +128,8 @@
     			</collision>
   		</link>
+		<gazebo reference="ptu_d46_tilt_link">
+        		<material>Gazebo/FlatBlack</material>
+        		<turnGravityOff>false</turnGravityOff>
+    		</gazebo>
 		<joint name="ptu_d46_tilt_joint" type="revolute">
     			<origin xyz="0 0 0.0455" rpy="1.5708 0 0" />

File: fsr_husky_description/urdf/parts/sick_lms100.urdf.xacro (robot description, xacro)
@@ -56,28 +56,37 @@
 			<origin xyz="${x} ${y} ${z}" rpy="${rx} ${ry} ${rz}" />
 		</joint>
-		<gazebo reference="laser">
-			<material value="Gazebo/Grey" />
- 			<sensor:ray name="laser">
-				<rayCount>1080</rayCount>
-				<rangeCount>1080</rangeCount>
-				<laserCount>1</laserCount>
-				<origin>0.0 0.0 0.0</origin>
-				<displayRays>false</displayRays>
-				<minAngle>-135</minAngle>
-				<maxAngle>135</maxAngle>
-				<minRange>0.5</minRange>
-				<maxRange>20.0</maxRange>
-				<resRange>0.01</resRange>
-				<updateRate>25.0</updateRate>
-				<controller:gazebo_ros_laser name="gazebo_ros_laser_controller" plugin="libgazebo_ros_laser.so">
-					<gaussianNoise>0.0042</gaussianNoise>
-					<alwaysOn>true</alwaysOn>
-					<updateRate>25.0</updateRate>
-					<topicName>scan</topicName>
-					<frameName>laser</frameName>
-					<interface:laser name="gazebo_ros_laser_iface" />
-      				</controller:gazebo_ros_laser>
-    			</sensor:ray>
- 		</gazebo>
+		<gazebo reference="sick_lms100">
+			<material>Gazebo/Grey</material>
+			<turnGravityOff>true</turnGravityOff>
+    			<sensor type="gpu_ray" name="sick_lms100">
+      				<pose>0 0 0 0 0 0</pose>
+      				<visualize>false</visualize>
+     	 			<update_rate>40</update_rate>
+      				<ray>
+        				<scan>
+          					<horizontal>
+            						<samples>720</samples>
+            						<resolution>1</resolution>
+            						<min_angle>-1.570796</min_angle>
+            						<max_angle>1.570796</max_angle>
+          					</horizontal>
+        				</scan>
+        				<range>
+          					<min>0.10</min>
+          					<max>30.0</max>
+          					<resolution>0.01</resolution>
+        				</range>
+        				<noise>
+          					<type>gaussian</type>
+          					<mean>0.0</mean>
+          					<stddev>0.01</stddev>
+        				</noise>
+      				</ray>
+      				<plugin name="gazebo_ros_head_hokuyo_controller" filename="libgazebo_ros_gpu_laser.so">
+        				<topicName>scan</topicName>
+        				<frameName>sick_lsm100</frameName>
+      				</plugin>
+    			</sensor>
+  		</gazebo>
 	</xacro:macro>
 </robot>
