Commit message: Major update to simulate the Husky in Gazebo

File: fsr_husky_description/urdf/arm/fsr_husky_arm.urdf.xacro (robot description, xacro)
@@ -135,8 +135,8 @@
       xyz="0 -1 0" />
     <limit
-      lower="-15708"
-      upper="15708"
-      effort="0"
-      velocity="0" />
+      lower="-1.5708"
+      upper="1.5708"
+      effort="100"
+      velocity="0.5" />
   </joint>
   <link
@@ -197,8 +197,8 @@
       xyz="0 1 0" />
     <limit
-      lower="-1"
-      upper="1"
-      effort="0"
-      velocity="0" />
+      lower="-0.5"
+      upper="0.25"
+      effort="20"
+      velocity="0.5" />
   </joint>
   <link
@@ -209,5 +209,5 @@
         rpy="0 0 0" />
       <mass
-        value="0.730115545526703" />
+	value="0.00001" /><!--value="0.730115545526703" />-->
       <inertia
         ixx="0.00564260404067653"
@@ -262,8 +262,8 @@
       xyz="0 0 -1" />
     <limit
-      lower="-1"
-      upper="1"
-      effort="0"
-      velocity="0" />
+      lower="-0.25"
+      upper="0.5"
+      effort="20"
+      velocity="0.5" />
   </joint>
   <link
@@ -274,5 +274,5 @@
         rpy="0 0 0" />
       <mass
-        value="12.099" />
+	value="0.00001" /><!--value="12.099" />-->
       <inertia
         ixx="0.060468"
@@ -383,9 +383,46 @@
       xyz="0 1 0" />
     <limit
-      lower="-1"
-      upper="1"
-      effort="0"
-      velocity="0" />
-  </joint>
+      lower="-0.5"
+      upper="0.25"
+      effort="20"
+      velocity="0.5" />
+  </joint>
+  <transmission name="upper_lift">
+    <type>transmission_interface/SimpleTransmission</type>
+    <joint name="upper_arm_joint"/>
+    <actuator name="upper_lift_motor">
+      <hardwareInterface>EffortJointInterface</hardwareInterface>
+      <mechanicalReduction>1</mechanicalReduction>
+    </actuator>
+  </transmission>
+  <transmission name="lower_lift">
+    <type>transmission_interface/SimpleTransmission</type>
+    <joint name="lower_arm_joint"/>
+    <actuator name="lower_lift_motor">
+      <hardwareInterface>EffortJointInterface</hardwareInterface>
+      <mechanicalReduction>1</mechanicalReduction>
+    </actuator>
+  </transmission>
+  <transmission name="mirror_lift">
+    <type>transmission_interface/SimpleTransmission</type>
+    <joint name="metal_detector_arm_joint"/>
+    <actuator name="mirror_lift_motor">
+      <hardwareInterface>EffortJointInterface</hardwareInterface>
+      <mechanicalReduction>1</mechanicalReduction>
+    </actuator>
+  </transmission>
+  <transmission name="sweep">
+    <type>transmission_interface/SimpleTransmission</type>
+    <joint name="arm_axel_joint"/>
+    <actuator name="sweep_motor">
+      <hardwareInterface>EffortJointInterface</hardwareInterface>
+      <mechanicalReduction>1</mechanicalReduction>
+    </actuator>
+  </transmission>
+  <gazebo>
+    <plugin name="gazebo_ros_control" filename="libgazebo_ros_control.so">
+      <robotNamespace>/arm</robotNamespace>
+    </plugin>
+  </gazebo>
 </xacro:macro>
 </robot>

File: fsr_husky_description/urdf/fsr_husky.urdf.xacro (robot description, xacro)
@@ -42,14 +42,14 @@
     xmlns:xacro="http://ros.org/wiki/xacro" name="husky">
     <!-- Included URDF/XACRO Files -->
-    <xacro:include filename="$(find husky_description)/urdf/materials.urdf.xacro" />
-    <xacro:include filename="$(find husky_description)/urdf/wheel.urdf.xacro" />
-    <xacro:include filename="$(find husky_description)/urdf/parts.urdf.xacro" />
-    <xacro:include filename="$(find fsr_husky_description)/urdf/parts/husky_bridge.urdf.xacro" />
-    <xacro:include filename="$(find fsr_husky_description)/urdf/parts/sick_lms100.urdf.xacro" />
-    <xacro:include filename="$(find fsr_husky_description)/urdf/parts/alfa_tube2h.urdf.xacro" />
-    <xacro:include filename="$(find fsr_husky_description)/urdf/parts/pointgrey_flea3.urdf.xacro" />
-    <xacro:include filename="$(find fsr_husky_description)/urdf/parts/gps_antenna.urdf.xacro" />
-    <xacro:include filename="$(find fsr_husky_description)/urdf/parts/ptu_d46.urdf.xacro" />
-    <xacro:include filename="$(find fsr_husky_description)/urdf/parts/mti.urdf.xacro" />
+    <xacro:include filename="$(find fsr_husky_description)/urdf/husky_parts/materials.urdf.xacro" />
+    <xacro:include filename="$(find fsr_husky_description)/urdf/husky_parts/wheel.urdf.xacro" />
+    <xacro:include filename="$(find fsr_husky_description)/urdf/husky_parts/parts.urdf.xacro" />
+    <xacro:include filename="$(find fsr_husky_description)/urdf/fsr_husky_parts/husky_bridge.urdf.xacro" />
+    <xacro:include filename="$(find fsr_husky_description)/urdf/fsr_husky_parts/sick_lms100.urdf.xacro" />
+    <xacro:include filename="$(find fsr_husky_description)/urdf/fsr_husky_parts/alfa_tube2h.urdf.xacro" />
+    <xacro:include filename="$(find fsr_husky_description)/urdf/fsr_husky_parts/pointgrey_flea3.urdf.xacro" />
+    <xacro:include filename="$(find fsr_husky_description)/urdf/fsr_husky_parts/gps_antenna.urdf.xacro" />
+    <xacro:include filename="$(find fsr_husky_description)/urdf/fsr_husky_parts/ptu_d46.urdf.xacro" />
+    <xacro:include filename="$(find fsr_husky_description)/urdf/fsr_husky_parts/mti.urdf.xacro" />
     <!-- PROPERTY LIST -->
     <!--All units in m-kg-s-radians unit system -->
@@ -76,5 +76,5 @@
     <!-- base_footprint is a fictitious link(frame) that is on the ground right below base_link origin, navigation stack depends on this frame -->
     <link name="base_footprint">
-        <inertial>
+        <!--<inertial>
             <mass value="0.0001" />
             <origin xyz="0 0 0" />
@@ -82,5 +82,5 @@
                 iyy="0.0001" iyz="0.0"
                 izz="0.0001" />
-        </inertial>
+	      </inertial>-->
         <visual>
             <origin xyz="0 0 0" rpy="0 0 0" />
@@ -91,5 +91,4 @@
     </link>
     <gazebo reference="base_footprint">
-        <material>Gazebo/Green</material>
         <turnGravityOff>false</turnGravityOff>
     </gazebo>
@@ -129,26 +128,10 @@
     </gazebo>
     <!-- WHEEL macros -->
-    <husky_wheel fb="back" lr="left" parent="base_link" translateX="-1" translateY="1" flipY="-1"/>
-    <husky_wheel fb="back" lr="right" parent="base_link" translateX="-1" translateY="-1" flipY="-1"/>
-    <husky_wheel fb="front" lr="left" parent="base_link" translateX="1" translateY="1" flipY="-1"/>
-    <husky_wheel fb="front" lr="right" parent="base_link" translateX="1" translateY="-1" flipY="-1"/>
-    <!-- BRIDGE macros -->
-    <husky_bridge prefix="front" parent="base_link" x="0.17" y="0" z="${base_z_size}" rx="0" ry="0" rz="0" />
-    <husky_bridge prefix="back" parent="base_link" x="-0.18" y="0" z="${base_z_size}" rx="0" ry="0" rz="0" />
-    <!-- MTi macro -->
-    <mti parent="back_husky_bridge" x="0" y="0" z="0.0" rx="0" ry="0" rz="0" />
-    <!-- CAMERA macros -->
-    <pointgrey_flea3 prefix="left" parent="front_husky_bridge" base_offset="-0.13" camera_offset="-0.05" camera_r="0" camera_p="0" camera_y="0" />
-    <pointgrey_flea3 prefix="right" parent="front_husky_bridge" base_offset="0.13" camera_offset="0.05" camera_r="0" camera_p="0" camera_y="0" />
-    <!-- PTU-D46 macro -->
-    <ptu_d46 parent="front_husky_bridge" x="0" y="-0.025" z="0" rx="0" ry="0" rz="1.5708" />
-    <!-- SICK macro -->
-    <sick_lms100 parent="ptu_d46_tilt_link" x="0.0" y="0.13" z="0.11" rx="0.0" ry="-0.7854" rz="-1.5708" />
-    <!-- GPS macro -->
-    <gps_antenna parent="back_husky_bridge" x="0" y="0.17" z="0.0" rx="0" ry="0" rz="0" />
+	<husky_wheel fb="back" lr="left" parent="base_link" translateX="-1" translateY="1" flipY="-1"/>
+	<husky_wheel fb="back" lr="right" parent="base_link" translateX="-1" translateY="-1" flipY="-1"/>
+	<husky_wheel fb="front" lr="left" parent="base_link" translateX="1" translateY="1" flipY="-1"/>
+	<husky_wheel fb="front" lr="right" parent="base_link" translateX="1" translateY="-1" flipY="-1"/>
     <!-- DECORATIONS -->
-    <!-- WiFi Antenna -->
-    <alfa_tube2h parent="back_husky_bridge" x="0" y="-0.17" z="0" rx="0" ry="0" rz="0" />
-   <!-- Top Plate -->
+    <!-- Top Plate -->
     <husky_part parent="base_footprint" name="top_plate" mesh="top_plate"
           colour="Yellow"
@@ -194,3 +177,20 @@
         </plugin>
     </gazebo>
+    <!-- FSR Husky Stuff -->
+    <!-- BRIDGE macros -->
+    <husky_bridge prefix="front" parent="base_link" x="0.17" y="0" z="${base_z_size}" rx="0" ry="0" rz="0" />
+    <husky_bridge prefix="back" parent="base_link" x="-0.18" y="0" z="${base_z_size}" rx="0" ry="0" rz="0" />
+    <!-- MTi macro -->
+    <mti parent="back_husky_bridge" x="0" y="0" z="0.0" rx="0" ry="0" rz="0" />
+    <!-- CAMERA macros -->
+    <pointgrey_flea3 prefix="left" parent="front_husky_bridge" base_offset="-0.13" camera_offset="-0.05" camera_r="0" camera_p="0" camera_y="0" />
+    <pointgrey_flea3 prefix="right" parent="front_husky_bridge" base_offset="0.13" camera_offset="0.05" camera_r="0" camera_p="0" camera_y="0" />
+    <!-- PTU-D46 macro -->
+    <ptu_d46 parent="front_husky_bridge" x="0" y="-0.025" z="0" rx="0" ry="0" rz="1.5708" />
+    <!-- SICK macro -->
+    <sick_lms100 parent="ptu_d46_tilt_link" x="0.0" y="0.13" z="0.11" rx="0.0" ry="-0.7854" rz="-1.5708" />
+    <!-- GPS macro -->
+    <gps_antenna parent="back_husky_bridge" x="0" y="0.17" z="0.0" rx="0" ry="0" rz="0" />
+    <!-- WiFi Antenna -->
+    <alfa_tube2h parent="back_husky_bridge" x="0" y="-0.17" z="0" rx="0" ry="0" rz="0" />
 </robot>

File: fsr_husky_description/urdf/fsr_husky_mine_detection.urdf.xacro (robot description, xacro)
@@ -42,13 +42,14 @@
     xmlns:xacro="http://ros.org/wiki/xacro" name="husky">
     <!-- Included URDF/XACRO Files -->
-    <xacro:include filename="$(find husky_description)/urdf/materials.urdf.xacro" />
-    <xacro:include filename="$(find husky_description)/urdf/wheel.urdf.xacro" />
-    <xacro:include filename="$(find husky_description)/urdf/parts.urdf.xacro" />
-    <xacro:include filename="$(find fsr_husky_description)/urdf/parts/husky_bridge.urdf.xacro" />
-    <xacro:include filename="$(find fsr_husky_description)/urdf/parts/sick_lms100.urdf.xacro" />
-    <xacro:include filename="$(find fsr_husky_description)/urdf/parts/alfa_tube2h.urdf.xacro" />
-    <xacro:include filename="$(find fsr_husky_description)/urdf/parts/pointgrey_flea3.urdf.xacro" />
-    <xacro:include filename="$(find fsr_husky_description)/urdf/parts/gps_antenna.urdf.xacro" />
-    <xacro:include filename="$(find fsr_husky_description)/urdf/parts/ptu_d46.urdf.xacro" />
+    <xacro:include filename="$(find fsr_husky_description)/urdf/husky_parts/materials.urdf.xacro" />
+    <xacro:include filename="$(find fsr_husky_description)/urdf/husky_parts/wheel.urdf.xacro" />
+    <xacro:include filename="$(find fsr_husky_description)/urdf/husky_parts/parts.urdf.xacro" />
+    <xacro:include filename="$(find fsr_husky_description)/urdf/fsr_husky_parts/husky_bridge.urdf.xacro" />
+    <xacro:include filename="$(find fsr_husky_description)/urdf/fsr_husky_parts/sick_lms100.urdf.xacro" />
+    <xacro:include filename="$(find fsr_husky_description)/urdf/fsr_husky_parts/alfa_tube2h.urdf.xacro" />
+    <xacro:include filename="$(find fsr_husky_description)/urdf/fsr_husky_parts/pointgrey_flea3.urdf.xacro" />
+    <xacro:include filename="$(find fsr_husky_description)/urdf/fsr_husky_parts/gps_antenna.urdf.xacro" />
+    <xacro:include filename="$(find fsr_husky_description)/urdf/fsr_husky_parts/ptu_d46.urdf.xacro" />
+    <xacro:include filename="$(find fsr_husky_description)/urdf/fsr_husky_parts/mti.urdf.xacro" />
     <xacro:include filename="$(find fsr_husky_description)/urdf/arm/fsr_husky_arm.urdf.xacro" />
     <!-- PROPERTY LIST -->
@@ -76,5 +77,5 @@
     <!-- base_footprint is a fictitious link(frame) that is on the ground right below base_link origin, navigation stack depends on this frame -->
     <link name="base_footprint">
-        <inertial>
+        <!--<inertial>
             <mass value="0.0001" />
             <origin xyz="0 0 0" />
@@ -82,5 +83,5 @@
                 iyy="0.0001" iyz="0.0"
                 izz="0.0001" />
-        </inertial>
+	      </inertial>-->
         <visual>
             <origin xyz="0 0 0" rpy="0 0 0" />
@@ -91,5 +92,4 @@
     </link>
     <gazebo reference="base_footprint">
-        <material>Gazebo/Green</material>
         <turnGravityOff>false</turnGravityOff>
     </gazebo>
@@ -113,5 +113,5 @@
             <origin xyz="0 0 0" rpy="0 0 0" />
             <geometry>
-                <mesh filename="package://husky_description/meshes/base_link.stl" />
+		<mesh filename="package://fsr_husky_description/models/husky_parts/base_link.stl" />
             </geometry>
             <material name="Black" />
@@ -129,10 +129,10 @@
     </gazebo>
     <!-- WHEEL macros -->
-    <husky_wheel fb="back" lr="left" parent="base_link" translateX="-1" translateY="1" flipY="-1"/>
-    <husky_wheel fb="back" lr="right" parent="base_link" translateX="-1" translateY="-1" flipY="-1"/>
-    <husky_wheel fb="front" lr="left" parent="base_link" translateX="1" translateY="1" flipY="-1"/>
-    <husky_wheel fb="front" lr="right" parent="base_link" translateX="1" translateY="-1" flipY="-1"/>
+	<husky_wheel fb="back" lr="left" parent="base_link" translateX="-1" translateY="1" flipY="-1"/>
+	<husky_wheel fb="back" lr="right" parent="base_link" translateX="-1" translateY="-1" flipY="-1"/>
+	<husky_wheel fb="front" lr="left" parent="base_link" translateX="1" translateY="1" flipY="-1"/>
+	<husky_wheel fb="front" lr="right" parent="base_link" translateX="1" translateY="-1" flipY="-1"/>
     <!-- DECORATIONS -->
-   <!-- Top Plate -->
+    <!-- Top Plate -->
     <husky_part parent="base_footprint" name="top_plate" mesh="top_plate"
           colour="Yellow"
@@ -141,5 +141,4 @@
     <gazebo reference="base_footprint_top_plate_part">
         <material>Gazebo/Yellow</material>
-	<turnGravityOff>false</turnGravityOff>
     </gazebo>
     <!-- User Rail -->
@@ -150,5 +149,4 @@
     <gazebo reference="base_footprint_user_rail_part">
         <material>Gazebo/Grey</material>
-	<turnGravityOff>false</turnGravityOff>
     </gazebo>
     <!-- Bumpers -->
@@ -159,5 +157,4 @@
     <gazebo reference="base_footprint_front_bumper_part">
         <material>Gazebo/FlatBlack</material>
-	<turnGravityOff>false</turnGravityOff>
     </gazebo>
     <husky_part parent="base_footprint" name="rear_bumper" mesh="bumper"
@@ -167,5 +164,4 @@
     <gazebo reference="base_footprint_rear_bumper_part">
         <material>Gazebo/FlatBlack</material>
-	<turnGravityOff>false</turnGravityOff>
     </gazebo>
     <gazebo>

File: fsr_husky_description/urdf/fsr_husky_parts/alfa_tube2h.urdf.xacro (robot description, xacro)
@@ -27,36 +27,62 @@
 	xmlns:controller="http://playerstage.sourceforge.net/gazebo/xmlschema/#controller"
 	xmlns:interface="http://playerstage.sourceforge.net/gazebo/xmlschema/#interface"
-	xmlns:xacro="http://ros.org/wiki/xacro" name="mti">
-	<xacro:include filename="$(find fsr_husky_description)/urdf/parts/common.xacro" />
-	<xacro:property name="mti_length" value="0.057" />
-	<xacro:property name="mti_width" value="0.042" />
-	<xacro:property name="mti_height" value="0.0235" />
-	<xacro:macro name="mti" params="parent x y z rx ry rz">
-  		<link name="base_imu">
-			<xacro:box_inertial x="${mti_length}"  y="${mti_width}" z="${mti_height}" mass="0.052" />
+	xmlns:xacro="http://ros.org/wiki/xacro" name="alfa_tube2h">
+	<!-- Alfa Tube 2H-->
+	<xacro:include filename="$(find fsr_husky_description)/urdf/fsr_husky_parts/common.xacro" />
+	<xacro:property name="alfa_length" value="0.132" />
+	<xacro:property name="alfa_radius" value="0.019" />
+	<xacro:property name="antenna_length" value="0.45" />
+	<xacro:property name="antenna_radius" value="0.008" />
+	<xacro:macro name="alfa_tube2h" params="parent x y z rx ry rz">
+  		<link name="alfa_tube2h">
+			<xacro:cylinder_inertial radius="${alfa_radius}" length="${alfa_length}" mass="0.100" />
 			<visual>
       				<geometry>
-        				<box size="${mti_length} ${mti_width} ${mti_height}"/>
+        				<cylinder length="${alfa_length}" radius="${alfa_radius}"/>
       				</geometry>
 				<origin rpy="0 0 0" xyz="0 0 0"/>
-      				<material name="Orange">
-        				<color rgba="1 0.4 0 1"/>
+      				<material name="White">
+        				<color rgba="1 1 1 1"/>
       				</material>
     			</visual>
     			<collision>
       				<geometry>
-        				<box size="${mti_length} ${mti_width} ${mti_height}"/>
+        				<cylinder length="${alfa_length}" radius="${alfa_radius}"/>
       				</geometry>
     			</collision>
   		</link>
-		<joint name="base_imu_joint" type="fixed">
-			<parent link="${parent}"/>
-			<child link="base_imu"/>
-			<origin xyz="${x} ${y} ${z+mti_height/2}" rpy="${rx} ${ry} ${rz}" />
-		</joint>
-		<gazebo reference="mti">
-        		<material>Gazebo/Orange</material>
+		<gazebo reference="alfa_tube2h">
+        		<material>Gazebo/White</material>
         		<turnGravityOff>false</turnGravityOff>
     		</gazebo>
+		<joint name="joint_alfa_tub2h" type="fixed">
+			<parent link="${parent}"/>
+			<child link="alfa_tube2h"/>
+			<origin xyz="${x} ${y} ${z+alfa_length/2}" rpy="${rx} ${ry} ${rz}" />
+		</joint>
+		<link name="wifi_antenna">
+			<xacro:cylinder_inertial radius="${antenna_radius}" length="${antenna_length}" mass="0.100" />
+			<visual>
+      				<geometry>
+        				<cylinder length="${antenna_length}" radius="${antenna_radius}"/>
+      				</geometry>
+				<origin rpy="0 0 0" xyz="0 0 0"/>
+      				<material name="White"/>
+    			</visual>
+    			<collision>
+      				<geometry>
+        				<cylinder length="${antenna_length}" radius="${antenna_radius}"/>
+      				</geometry>
+    			</collision>
+  		</link>
+		<gazebo reference="wifi_antenna">
+        		<material>Gazebo/White</material>
+        		<turnGravityOff>false</turnGravityOff>
+    		</gazebo>
+		<joint name="joint_wifi_anetnna" type="fixed">
+			<parent link="alfa_tube2h"/>
+			<child link="wifi_antenna"/>
+			<origin xyz="0 0 ${alfa_length/2+antenna_length/2}" rpy="0 0 0" />
+		</joint>
 	</xacro:macro>
 </robot>

File: fsr_husky_description/urdf/fsr_husky_parts/gps_antenna.urdf.xacro (robot description, xacro)
@@ -29,5 +29,5 @@
 	xmlns:xacro="http://ros.org/wiki/xacro" name="gps_antenna">
 	<!-- GPS Antenna -->
-	<xacro:include filename="$(find fsr_husky_description)/urdf/parts/common.xacro" />
+	<xacro:include filename="$(find fsr_husky_description)/urdf/fsr_husky_parts/common.xacro" />
 	<xacro:property name="alfa_length" value="0.132" />
 	<xacro:property name="alfa_radius" value="0.019" />
@@ -50,5 +50,5 @@
       				<origin xyz="-0.035 0 0" rpy="1.5708 0 0" />
       				<geometry>
-        				<mesh filename="package://fsr_husky_description/models/gps_antenna.stl" />
+					<mesh filename="package://fsr_husky_description/models/fsr_husky_parts/gps_antenna.stl" />
       				</geometry>
       				<material name="White">
@@ -59,12 +59,8 @@
       				<origin xyz="-0.035 0 0" rpy="1.5708 0 0" />
       				<geometry>
-        				<mesh filename="package://fsr_husky_description/models/gps_antenna.stl" />
+					<mesh filename="package://fsr_husky_description/models/fsr_husky_parts/gps_antenna.stl" />
      			 	</geometry>
     			</collision>
   		</link>
-		<gazebo reference="gps_antenna">
-        		<material>Gazebo/White</material>
-        		<turnGravityOff>false</turnGravityOff>
-    		</gazebo>
 		<joint name="gps_anetnna_joint" type="fixed">
 			<parent link="${parent}"/>
@@ -72,4 +68,20 @@
 			<origin xyz="${x} ${y} ${z}" rpy="${rx} ${ry} ${rz}" />
 		</joint>
+		<gazebo reference="gps_antenna">
+        		<material>Gazebo/White</material>
+        		<turnGravityOff>false</turnGravityOff>
+		</gazebo>
+		<gazebo>
+			<plugin name="gazebo_ros_gps" filename="libhector_gazebo_ros_gps.so">
+			  <updateRate>4.0</updateRate>
+			  <bodyName>gps_antenna</bodyName>
+			  <topicName>fix</topicName>
+			  <velocityTopicName>fix_velocity</velocityTopicName>
+			  <drift>1.0 1.0 1.0</drift>
+			  <gaussianNoise>0.01 0.01 0.01</gaussianNoise>
+			  <velocityDrift>0 0 0</velocityDrift>
+			  <velocityGaussianNoise>0.05 0.05 0.05</velocityGaussianNoise>
+			</plugin>
+    		</gazebo>
 	</xacro:macro>
 </robot>

File: fsr_husky_description/urdf/fsr_husky_parts/husky_bridge.urdf.xacro (robot description, xacro)
@@ -46,5 +46,5 @@
       				<origin xyz="-0.12511 0 ${-bridge_height}" rpy="1.5708 0 1.5708" />
       				<geometry>
-        				<mesh filename="package://fsr_husky_description/models/bridge.stl" />
+					<mesh filename="package://fsr_husky_description/models/fsr_husky_parts/bridge.stl" />
       				</geometry>
       				<material name="Gray" />
@@ -53,5 +53,5 @@
       				<origin xyz="-0.12511 0 ${-bridge_height}" rpy="1.5708 0 1.5708" />
       				<geometry>
-        				<mesh filename="package://fsr_husky_description/models/bridge.stl" />
+					<mesh filename="package://fsr_husky_description/models/fsr_husky_parts/bridge.stl" />
       				</geometry>
     			</collision>
