Commit message: Major update to simulate the Husky in Gazebo

File: fsr_husky_description/urdf/fsr_husky_parts/mti.urdf.xacro (robot description, xacro)
@@ -27,62 +27,46 @@
 	xmlns:controller="http://playerstage.sourceforge.net/gazebo/xmlschema/#controller"
 	xmlns:interface="http://playerstage.sourceforge.net/gazebo/xmlschema/#interface"
-	xmlns:xacro="http://ros.org/wiki/xacro" name="alfa_tube2h">
-	<!-- Alfa Tube 2H-->
-	<xacro:include filename="$(find fsr_husky_description)/urdf/parts/common.xacro" />
-	<xacro:property name="alfa_length" value="0.132" />
-	<xacro:property name="alfa_radius" value="0.019" />
-	<xacro:property name="antenna_length" value="0.45" />
-	<xacro:property name="antenna_radius" value="0.008" />
-	<xacro:macro name="alfa_tube2h" params="parent x y z rx ry rz">
-  		<link name="alfa_tube2h">
-			<xacro:cylinder_inertial radius="${alfa_radius}" length="${alfa_length}" mass="0.100" />
+	xmlns:xacro="http://ros.org/wiki/xacro" name="mti">
+	<xacro:include filename="$(find fsr_husky_description)/urdf/fsr_husky_parts/common.xacro" />
+	<xacro:property name="mti_length" value="0.057" />
+	<xacro:property name="mti_width" value="0.042" />
+	<xacro:property name="mti_height" value="0.0235" />
+	<xacro:macro name="mti" params="parent x y z rx ry rz">
+  		<link name="base_imu">
+			<xacro:box_inertial x="${mti_length}"  y="${mti_width}" z="${mti_height}" mass="0.052" />
 			<visual>
       				<geometry>
-        				<cylinder length="${alfa_length}" radius="${alfa_radius}"/>
+        				<box size="${mti_length} ${mti_width} ${mti_height}"/>
       				</geometry>
 				<origin rpy="0 0 0" xyz="0 0 0"/>
-      				<material name="White">
-        				<color rgba="1 1 1 1"/>
+      				<material name="Orange">
+        				<color rgba="1 0.4 0 1"/>
       				</material>
     			</visual>
     			<collision>
       				<geometry>
-        				<cylinder length="${alfa_length}" radius="${alfa_radius}"/>
+        				<box size="${mti_length} ${mti_width} ${mti_height}"/>
       				</geometry>
     			</collision>
   		</link>
-		<gazebo reference="alfa_tube2h">
-        		<material>Gazebo/White</material>
+		<joint name="base_imu_joint" type="fixed">
+			<parent link="${parent}"/>
+			<child link="base_imu"/>
+			<origin xyz="${x} ${y} ${z+mti_height/2}" rpy="${rx} ${ry} ${rz}" />
+		</joint>
+		<gazebo reference="base_imu">
+        		<material>Gazebo/Orange</material>
         		<turnGravityOff>false</turnGravityOff>
     		</gazebo>
-		<joint name="joint_alfa_tub2h" type="fixed">
-			<parent link="${parent}"/>
-			<child link="alfa_tube2h"/>
-			<origin xyz="${x} ${y} ${z+alfa_length/2}" rpy="${rx} ${ry} ${rz}" />
-		</joint>
-		<link name="wifi_antenna">
-			<xacro:cylinder_inertial radius="${antenna_radius}" length="${antenna_length}" mass="0.100" />
-			<visual>
-      				<geometry>
-        				<cylinder length="${antenna_length}" radius="${antenna_radius}"/>
-      				</geometry>
-				<origin rpy="0 0 0" xyz="0 0 0"/>
-      				<material name="White"/>
-    			</visual>
-    			<collision>
-      				<geometry>
-        				<cylinder length="${antenna_length}" radius="${antenna_radius}"/>
-      				</geometry>
-    			</collision>
-  		</link>
-		<gazebo reference="wifi_antenna">
-        		<material>Gazebo/White</material>
-        		<turnGravityOff>false</turnGravityOff>
-    		</gazebo>
-		<joint name="joint_wifi_anetnna" type="fixed">
-			<parent link="alfa_tube2h"/>
-			<child link="wifi_antenna"/>
-			<origin xyz="0 0 ${alfa_length/2+antenna_length/2}" rpy="0 0 0" />
-		</joint>
+		<gazebo>
+		    <plugin name="gazebo_ros_imu" filename="libgazebo_ros_imu.so">
+			<alwaysOn>true</alwaysOn>
+			<bodyName>base_imu</bodyName>
+			<topicName>imu_data</topicName>
+			<serviceName>imu_service</serviceName>
+			<gaussianNoise>0.0</gaussianNoise>
+			<updateRate>30.0</updateRate>
+		    </plugin>
+		</gazebo>
 	</xacro:macro>
 </robot>

File: fsr_husky_description/urdf/fsr_husky_parts/pointgrey_flea3.urdf.xacro (robot description, xacro)
@@ -29,5 +29,5 @@
 	xmlns:xacro="http://ros.org/wiki/xacro" name="pointgrey_flea3">
 	<!-- PointGrey Flea 3 -->
-	<xacro:include filename="$(find fsr_husky_description)/urdf/parts/common.xacro" />
+	<xacro:include filename="$(find fsr_husky_description)/urdf/fsr_husky_parts/common.xacro" />
 	<xacro:property name="base_x" value="0.040" />
 	<xacro:property name="base_y" value="0.150" />

File: fsr_husky_description/urdf/fsr_husky_parts/ptu_d46.urdf.xacro (robot description, xacro)
@@ -45,5 +45,5 @@
       				<origin xyz="0 0 0" rpy="0 0 0" />
       				<geometry>
-        				<mesh filename="package://fsr_husky_description/models/ptu_d46_base_link.stl" />
+					<mesh filename="package://fsr_husky_description/models/fsr_husky_parts/ptu_d46_base_link.stl" />
      	 			</geometry>
       				<material name="DarkGray" />
@@ -52,5 +52,5 @@
       				<origin xyz="0 0 0" rpy="0 0 0" />
       				<geometry>
-        				<mesh filename="package://fsr_husky_description/models/ptu_d46_base_link.stl" />
+					<mesh filename="package://fsr_husky_description/models/fsr_husky_parts/ptu_d46_base_link.stl" />
       				</geometry>
     			</collision>
@@ -80,5 +80,5 @@
       				<origin xyz="0 0 0" rpy="0 0 0" />
       				<geometry>
-        				<mesh filename="package://fsr_husky_description/models/ptu_d46_pan_link.stl" />
+					<mesh filename="package://fsr_husky_description/models/fsr_husky_parts/ptu_d46_pan_link.stl" />
       				</geometry>
       				<material name="DarkGray" />
@@ -87,5 +87,5 @@
       				<origin xyz="0 0 0" rpy="0 0 0" />
       				<geometry>
-					<mesh filename="package://fsr_husky_description/models/ptu_d46_pan_link.stl" />
+					<mesh filename="package://fsr_husky_description/models/fsr_husky_parts/ptu_d46_pan_link.stl" />
       				</geometry>
     			</collision>
@@ -100,5 +100,6 @@
     			<child link="ptu_d46_pan_link" />
     			<axis xyz="0 0 -1" />
-    			<limit effort="0" lower="-0.5" upper="0.5" velocity="0" />
+    			<limit effort="6.0" lower="-0.5" upper="0.5" velocity="0.5" />
+			<dynamics damping="0.008" friction="0.6" />
   		</joint>
 		<link name="ptu_d46_tilt_link">
@@ -117,5 +118,5 @@
       				<origin xyz="0 0 0" rpy="0 0 0" />
       				<geometry>
-        				<mesh filename="package://fsr_husky_description/models/ptu_d46_tilt_link.stl" />
+					<mesh filename="package://fsr_husky_description/models/fsr_husky_parts/ptu_d46_tilt_link.stl" />
       				</geometry>
       				<material name="DarkGray" />
@@ -124,5 +125,5 @@
       				<origin xyz="0 0 0" rpy="0 0 0" />
       				<geometry>
-        				<mesh filename="package://fsr_husky_description/models/ptu_d46_tilt_link.stl" />
+					<mesh filename="package://fsr_husky_description/models/fsr_husky_parts/ptu_d46_tilt_link.stl" />
       				</geometry>
     			</collision>
@@ -137,6 +138,28 @@
     			<child link="ptu_d46_tilt_link" />
     			<axis xyz="-1 0 0" />
-    			<limit effort="0" lower="-0.5" upper="0.5" velocity="0" />
+    			<limit effort="6.0" lower="-0.5" upper="0.5" velocity="0.5" />
+			<dynamics damping="0.008" friction="0.6" />
   		</joint>
+		<transmission name="pan">
+		  <type>transmission_interface/SimpleTransmission</type>
+		  <joint name="ptu_d46_pan_joint"/>
+		  <actuator name="pan_motor">
+		    <hardwareInterface>EffortJointInterface</hardwareInterface>
+		    <mechanicalReduction>1</mechanicalReduction>
+		  </actuator>
+		</transmission>
+		<transmission name="tilt">
+		  <type>transmission_interface/SimpleTransmission</type>
+		  <joint name="ptu_d46_tilt_joint"/>
+		  <actuator name="tilt_motor">
+		    <hardwareInterface>EffortJointInterface</hardwareInterface>
+		    <mechanicalReduction>1</mechanicalReduction>
+		  </actuator>
+		</transmission>
+		<gazebo>
+		  <plugin name="gazebo_ros_control" filename="libgazebo_ros_control.so">
+		    <robotNamespace>/ptu_d46</robotNamespace>
+		  </plugin>
+		</gazebo>
 	</xacro:macro>
 </robot>

File: fsr_husky_description/urdf/fsr_husky_parts/sick_lms100.urdf.xacro (robot description, xacro)
@@ -29,5 +29,5 @@
 	xmlns:xacro="http://ros.org/wiki/xacro" name="sick_lms100">
 	<!-- SICK LMS100-->
-	<xacro:include filename="$(find fsr_husky_description)/urdf/parts/common.xacro" />
+	<xacro:include filename="$(find fsr_husky_description)/urdf/fsr_husky_parts/common.xacro" />
 	<xacro:property name="laser_x" value="0.105" />
 	<xacro:property name="laser_y" value="0.102" />
@@ -40,5 +40,5 @@
 				<origin xyz="0 0 0" rpy="0 0 0" />
 				<geometry>
-					<mesh filename="package://fsr_husky_description/models/sick_lms100.stl" />
+					<mesh filename="package://fsr_husky_description/models/fsr_husky_parts/sick_lms100.stl" />
 				</geometry>
 				<material name="DarkGray" />
@@ -46,5 +46,5 @@
     			<collision>
       				<geometry>
-        				<mesh filename="package://fsr_husky_description/models/sick_lms100.stl" />
+					<mesh filename="package://fsr_husky_description/models/fsr_husky_parts/sick_lms100.stl" />
         				<!-- <box size="${laser_x} ${laser_y} ${laser_z}" /> -->
       				</geometry>
@@ -80,10 +80,10 @@
           					<type>gaussian</type>
           					<mean>0.0</mean>
-          					<stddev>0.01</stddev>
+          					<stddev>0.001</stddev>
         				</noise>
       				</ray>
-      				<plugin name="gazebo_ros_head_hokuyo_controller" filename="libgazebo_ros_gpu_laser.so">
+      				<plugin name="gazebo_ros_laser" filename="libgazebo_ros_gpu_laser.so">
         				<topicName>scan</topicName>
-        				<frameName>sick_lsm100</frameName>
+        				<frameName>sick_lms100</frameName>
       				</plugin>
     			</sensor>

Commit message: Major update.

File: fsr_husky_description/urdf/arm/fsr_husky_arm.urdf.xacro (robot description, xacro)
@@ -274,5 +274,5 @@
         rpy="0 0 0" />
       <mass
-	value="0.00001" /><!--value="12.099" />-->
+	value="12.099" />
       <inertia
         ixx="0.060468"
@@ -323,4 +323,43 @@
     <axis
       xyz="0 0 0" />
+  </joint>
+  <link name="left_coil">
+      <visual>
+          <origin xyz="0 0 0" rpy="0 0 0" />
+          <geometry>
+              <box size="0.001 0.001 0.001" />
+          </geometry>
+      </visual>
+  </link>
+  <joint name="left_coil_joint" type="fixed">
+      <origin xyz="0.18 0 0" rpy="0 0 0" />
+      <parent link="metal_detector_antenna"/>
+      <child link="left_coil" />
+  </joint>
+  <link name="middle_coil">
+      <visual>
+          <origin xyz="0 0 0" rpy="0 0 0" />
+          <geometry>
+              <box size="0.001 0.001 0.001" />
+          </geometry>
+      </visual>
+  </link>
+  <joint name="middle_coil_joint" type="fixed">
+      <origin xyz="0 0 0" rpy="0 0 0" />
+      <parent link="metal_detector_antenna"/>
+      <child link="middle_coil" />
+  </joint>
+  <link name="right_coil">
+      <visual>
+          <origin xyz="0 0 0" rpy="0 0 0" />
+          <geometry>
+              <box size="0.001 0.001 0.001" />
+          </geometry>
+      </visual>
+  </link>
+  <joint name="right_coil_joint" type="fixed">
+      <origin xyz="-0.18 0 0" rpy="0 0 0" />
+      <parent link="metal_detector_antenna"/>
+      <child link="right_coil" />
   </joint>
   <link
@@ -388,16 +427,16 @@
       velocity="0.5" />
   </joint>
-  <transmission name="upper_lift">
+  <transmission name="lift">
     <type>transmission_interface/SimpleTransmission</type>
     <joint name="upper_arm_joint"/>
-    <actuator name="upper_lift_motor">
+    <actuator name="lift_motor">
       <hardwareInterface>EffortJointInterface</hardwareInterface>
       <mechanicalReduction>1</mechanicalReduction>
     </actuator>
   </transmission>
-  <transmission name="lower_lift">
+  <transmission name="mimic_lift">
     <type>transmission_interface/SimpleTransmission</type>
     <joint name="lower_arm_joint"/>
-    <actuator name="lower_lift_motor">
+    <actuator name="mimic_lift_motor">
       <hardwareInterface>EffortJointInterface</hardwareInterface>
       <mechanicalReduction>1</mechanicalReduction>
@@ -421,7 +460,16 @@
   </transmission>
   <gazebo>
-    <plugin name="gazebo_ros_control" filename="libgazebo_ros_control.so">
-      <robotNamespace>/arm</robotNamespace>
-    </plugin>
+	<plugin name="mimic_plugin1" filename="libmimic_plugin.so">
+            <joint>upper_arm_joint</joint>
+            <mimicJoint>lower_arm_joint</mimicJoint>
+            <multiplier>1.0</multiplier>
+        </plugin>
+  </gazebo>
+  <gazebo>
+	<plugin name="mimic_plugin2" filename="libmimic_plugin.so">
+            <joint>upper_arm_joint</joint>
+            <mimicJoint>metal_detector_arm_joint</mimicJoint>
+            <multiplier>-1.0</multiplier>
+        </plugin>
   </gazebo>
 </xacro:macro>

File: fsr_husky_description/urdf/fsr_husky.urdf.xacro (robot description, xacro)
@@ -24,6 +24,6 @@
 (INCLUDING NEGLIGENCE OR OTHERWISE) ARISING IN ANY WAY OUT OF THE USE OF THIS
 SOFTWARE, EVEN IF ADVISED OF THE POSSIBILITY OF SUCH DAMAGE.
-This program contains the description of the robot base model for the Clearpath
-Husky A200 modified by the ISR University of Coimbra
+This program contains the description of the HRATC2014 Husky robot based on the original Clearpath
+Husky A200 file and modified by the ISR University of Coimbra
 -->
 <robot
@@ -52,4 +52,5 @@
     <xacro:include filename="$(find fsr_husky_description)/urdf/fsr_husky_parts/ptu_d46.urdf.xacro" />
     <xacro:include filename="$(find fsr_husky_description)/urdf/fsr_husky_parts/mti.urdf.xacro" />
+    <xacro:include filename="$(find fsr_husky_description)/urdf/arm/fsr_husky_arm.urdf.xacro" />
     <!-- PROPERTY LIST -->
     <!--All units in m-kg-s-radians unit system -->
@@ -112,5 +113,5 @@
             <origin xyz="0 0 0" rpy="0 0 0" />
             <geometry>
-                <mesh filename="package://husky_description/meshes/base_link.stl" />
+		<mesh filename="package://fsr_husky_description/models/husky_parts/base_link.stl" />
             </geometry>
             <material name="Black" />
@@ -165,6 +166,6 @@
     </gazebo>
     <gazebo>
-	    <plugin name="husky_diff_controller" filename="libhusky_gazebo_plugins.so">
-		    <alwaysOn>true</alwaysOn>
+	<plugin name="husky_diff_controller" filename="libhusky_gazebo_plugins.so">
+	    <alwaysOn>true</alwaysOn>
             <updateRate>100.0</updateRate>
             <backLeftJoint>joint_back_left_wheel</backLeftJoint>
@@ -184,6 +185,6 @@
     <mti parent="back_husky_bridge" x="0" y="0" z="0.0" rx="0" ry="0" rz="0" />
     <!-- CAMERA macros -->
-    <pointgrey_flea3 prefix="left" parent="front_husky_bridge" base_offset="-0.13" camera_offset="-0.05" camera_r="0" camera_p="0" camera_y="0" />
-    <pointgrey_flea3 prefix="right" parent="front_husky_bridge" base_offset="0.13" camera_offset="0.05" camera_r="0" camera_p="0" camera_y="0" />
+    <pointgrey_flea3 prefix="right" parent="front_husky_bridge" base_offset="-0.13" camera_offset="-0.05" camera_r="0" camera_p="0" camera_y="0" />
+    <pointgrey_flea3 prefix="left" parent="front_husky_bridge" base_offset="0.13" camera_offset="0.05" camera_r="0" camera_p="0" camera_y="0" />
     <!-- PTU-D46 macro -->
     <ptu_d46 parent="front_husky_bridge" x="0" y="-0.025" z="0" rx="0" ry="0" rz="1.5708" />
@@ -194,3 +195,8 @@
     <!-- WiFi Antenna -->
     <alfa_tube2h parent="back_husky_bridge" x="0" y="-0.17" z="0" rx="0" ry="0" rz="0" />
+    <gazebo>
+      <plugin name="gazebo_ros_control" filename="libgazebo_ros_control.so">
+	<!--<robotNamespace>/husky</robotNamespace>-->
+      </plugin>
+    </gazebo>
 </robot>

File: fsr_husky_description/urdf/fsr_husky_mine_detection.urdf.xacro (robot description, xacro)
@@ -24,6 +24,6 @@
 (INCLUDING NEGLIGENCE OR OTHERWISE) ARISING IN ANY WAY OUT OF THE USE OF THIS
 SOFTWARE, EVEN IF ADVISED OF THE POSSIBILITY OF SUCH DAMAGE.
-This program contains the description of the robot base model for the Clearpath
-Husky A200 modified by the ISR University of Coimbra
+This program contains the description of the HRATC2014 Husky robot based on the original Clearpath
+Husky A200 file and modified by the ISR University of Coimbra
 -->
 <robot
@@ -118,7 +118,8 @@
         </visual>
 		<collision>
-			<origin xyz="0 0 ${wheel_x_size/2 - base_z_origin_to_wheel_origin - 0.02}" rpy="0 0 0 " />
+			<!--<origin xyz="0 0 ${wheel_x_size/2 - base_z_origin_to_wheel_origin - 0.02}" rpy="0 0 0 " />-->
 			<geometry>
-				<box size = "${base_x_size+0.02} ${base_y_size} ${base_z_size + 0.02}"/> <!--making it slightly bigger in x and z direction-->
+				<mesh filename="package://fsr_husky_description/models/husky_parts/base_link.stl" />
+				<!--<box size = "${base_x_size+0.02} ${base_y_size} ${base_z_size + 0.02}"/>--> <!--making it slightly bigger in x and z direction-->
 			</geometry>
 		</collision>
@@ -175,5 +176,5 @@
             <wheelSeparation>${base_y_size}</wheelSeparation>
             <wheelDiameter>${wheel_x_size}</wheelDiameter>
-            <torque>35</torque>
+            <torque>50</torque>
         </plugin>
     </gazebo>
@@ -185,6 +186,6 @@
     <mti parent="back_husky_bridge" x="0" y="0" z="0.0" rx="0" ry="0" rz="0" />
     <!-- CAMERA macros -->
-    <pointgrey_flea3 prefix="left" parent="front_husky_bridge" base_offset="-0.13" camera_offset="-0.05" camera_r="0" camera_p="0" camera_y="0" />
-    <pointgrey_flea3 prefix="right" parent="front_husky_bridge" base_offset="0.13" camera_offset="0.05" camera_r="0" camera_p="0" camera_y="0" />
+    <pointgrey_flea3 prefix="right" parent="front_husky_bridge" base_offset="-0.13" camera_offset="-0.05" camera_r="0" camera_p="0" camera_y="0" />
+    <pointgrey_flea3 prefix="left" parent="front_husky_bridge" base_offset="0.13" camera_offset="0.05" camera_r="0" camera_p="0" camera_y="0" />
     <!-- PTU-D46 macro -->
     <ptu_d46 parent="front_husky_bridge" x="0" y="-0.025" z="0" rx="0" ry="0" rz="1.5708" />
@@ -197,3 +198,8 @@
     <!-- FSR Husky De-mining Arm -->
     <fsr_husky_arm parent="base_link" x="0.120" y="-0.15" z="${base_z_size}" rx="0" ry="0" rz="0" />
+    <gazebo>
+      <plugin name="gazebo_ros_control" filename="libgazebo_ros_control.so">
+	<!--<robotNamespace>/husky</robotNamespace>-->
+      </plugin>
+    </gazebo>
 </robot>

File: fsr_husky_description/urdf/fsr_husky_parts/common.xacro (robot description, xacro)
@@ -1,3 +1,27 @@
 <?xml version="1.0"?>
+<!--
+Copyright (c) 2013, Goncalo Cabrita, ISR University of Coimbra
+All rights reserved.
+Redistribution and use in source and binary forms, with or without
+modification, are permitted provided that the following conditions are met:
+    * Redistributions of source code must retain the above copyright
+      notice, this list of conditions and the following disclaimer.
+    * Redistributions in binary form must reproduce the above copyright
+      notice, this list of conditions and the following disclaimer in the
+      documentation and/or other materials provided with the distribution.
+    * Neither the name of Clearpath Robotics nor the
+      names of its contributors may be used to endorse or promote products
+      derived from this software without specific prior written permission.
+THIS SOFTWARE IS PROVIDED BY THE COPYRIGHT HOLDERS AND CONTRIBUTORS "AS IS" AND
+ANY EXPRESS OR IMPLIED WARRANTIES, INCLUDING, BUT NOT LIMITED TO, THE IMPLIED
+WARRANTIES OF MERCHANTABILITY AND FITNESS FOR A PARTICULAR PURPOSE ARE
+DISCLAIMED. IN NO EVENT SHALL THE COPYRIGHT HOLDERS BE LIABLE FOR ANY
+DIRECT, INDIRECT, INCIDENTAL, SPECIAL, EXEMPLARY, OR CONSEQUENTIAL DAMAGES
+(INCLUDING, BUT NOT LIMITED TO, PROCUREMENT OF SUBSTITUTE GOODS OR SERVICES;
+LOSS OF USE, DATA, OR PROFITS; OR BUSINESS INTERRUPTION) HOWEVER CAUSED AND
+ON ANY THEORY OF LIABILITY, WHETHER IN CONTRACT, STRICT LIABILITY, OR TORT
+(INCLUDING NEGLIGENCE OR OTHERWISE) ARISING IN ANY WAY OUT OF THE USE OF THIS
+SOFTWARE, EVEN IF ADVISED OF THE POSSIBILITY OF SUCH DAMAGE.
+-->
 <robot
   xmlns:xacro="http://ros.org/wiki/xacro">

File: fsr_husky_description/urdf/fsr_husky_parts/gps_antenna.urdf.xacro (robot description, xacro)
@@ -76,6 +76,6 @@
 			  <updateRate>4.0</updateRate>
 			  <bodyName>gps_antenna</bodyName>
-			  <topicName>fix</topicName>
-			  <velocityTopicName>fix_velocity</velocityTopicName>
+			  <topicName>/gps/fix</topicName>
+			  <velocityTopicName>/gps/fix_velocity</velocityTopicName>
 			  <drift>1.0 1.0 1.0</drift>
 			  <gaussianNoise>0.01 0.01 0.01</gaussianNoise>

File: fsr_husky_description/urdf/fsr_husky_parts/mti.urdf.xacro (robot description, xacro)
@@ -63,5 +63,5 @@
 			<alwaysOn>true</alwaysOn>
 			<bodyName>base_imu</bodyName>
-			<topicName>imu_data</topicName>
+			<topicName>/imu/data</topicName>
 			<serviceName>imu_service</serviceName>
 			<gaussianNoise>0.0</gaussianNoise>

File: fsr_husky_description/urdf/fsr_husky_parts/pointgrey_flea3.urdf.xacro (robot description, xacro)
@@ -112,5 +112,5 @@
 			<parent link="${prefix}_camera_standoff"/>
 			<child link="${prefix}_camera"/>
-			<origin xyz="0 0 ${standoff_length/2+flea_size/2}" rpy="${camera_r} ${1.5708+camera_p} ${camera_y}" />
+			<origin xyz="0 0 ${standoff_length/2+flea_size/2}" rpy="${camera_r} ${camera_p} ${camera_y}" />
 		</joint>
 		<!-- Camera Lense -->
@@ -121,5 +121,5 @@
         				<cylinder length="${lense_length}" radius="${lense_radius}"/>
       				</geometry>
-				<origin rpy="0 0 0" xyz="0 0 0"/>
+				<origin rpy="0 1.57 0" xyz="0 0 -0.035"/>
       				<material name="Black"/>
     			</visual>

File: fsr_husky_description/urdf/fsr_husky_parts/ptu_d46.urdf.xacro (robot description, xacro)
@@ -134,5 +134,5 @@
     		</gazebo>
 		<joint name="ptu_d46_tilt_joint" type="revolute">
-    			<origin xyz="0 0 0.0455" rpy="1.5708 0 0" />
+    			<origin xyz="0 0 0.0455" rpy="1.3 0 0" />
     			<parent link="ptu_d46_pan_link" />
     			<child link="ptu_d46_tilt_link" />
@@ -157,9 +157,9 @@
 		  </actuator>
 		</transmission>
-		<gazebo>
+		<!--<gazebo>
 		  <plugin name="gazebo_ros_control" filename="libgazebo_ros_control.so">
 		    <robotNamespace>/ptu_d46</robotNamespace>
 		  </plugin>
-		</gazebo>
+		</gazebo>-->
 	</xacro:macro>
 </robot>

File: fsr_husky_description/urdf/fsr_husky_parts/sick_lms100.urdf.xacro (robot description, xacro)
@@ -59,5 +59,5 @@
 			<material>Gazebo/Grey</material>
 			<turnGravityOff>true</turnGravityOff>
-    			<sensor type="gpu_ray" name="sick_lms100">
+    			<sensor type="ray" name="sick_lms100">
       				<pose>0 0 0 0 0 0</pose>
       				<visualize>false</visualize>
@@ -83,5 +83,5 @@
         				</noise>
       				</ray>
-      				<plugin name="gazebo_ros_laser" filename="libgazebo_ros_gpu_laser.so">
+      				<plugin name="gazebo_ros_laser" filename="libgazebo_ros_laser.so">
         				<topicName>scan</topicName>
         				<frameName>sick_lms100</frameName>
