Commit message: Major update to the fsr_husky framework.

File: fsr_husky_description/urdf/arm/fsr_husky_arm.urdf.xacro (robot description, xacro)
@@ -30,26 +30,26 @@
 <xacro:macro name="fsr_husky_arm" params="parent x y z rx ry rz">
   <link
-    name="base_arm_link">
-    <inertial>
-      <origin
-        xyz="0.0748500402726595 0.0136470618219005 -0.0925164110070736"
-        rpy="0 0 0" />
-      <mass
-        value="0.215286927386896" />
-      <inertia
-        ixx="0.00151952875960782"
-        ixy="-5.00239624175035E-05"
-        ixz="-0.000104007201846032"
-        iyy="0.00181155299285244"
-        iyz="0.000216578123822788"
-        izz="0.000582288664758318" />
-    </inertial>
-    <visual>
-      <origin
-        xyz="0 0 0"
-        rpy="0 0 0" />
-      <geometry>
-        <mesh
-          filename="package://fsr_husky_description/models/arm/base_arm_link.STL" />
+    name="arm_base_link">
+    <inertial>
+      <origin
+        xyz="-0.1981 0.35759 0.20723"
+        rpy="0 0 0" />
+      <mass
+        value="1.1522" />
+      <inertia
+        ixx="0.011095"
+        ixy="0.0012342"
+        ixz="0.00013298"
+        iyy="0.0047097"
+        iyz="0.00037003"
+        izz="0.013904" />
+    </inertial>
+    <visual>
+      <origin
+        xyz="0 0 0"
+        rpy="0 0 0" />
+      <geometry>
+        <mesh
+          filename="package://fsr_husky_description/models/arm/arm_base_link.STL" />
       </geometry>
       <material
@@ -65,40 +65,36 @@
       <geometry>
         <mesh
-          filename="package://fsr_husky_description/models/arm/base_arm_link.STL" />
-      </geometry>
-    </collision>
-  </link>
-  <gazebo reference="base_arm_link">
+          filename="package://fsr_husky_description/models/arm/arm_base_link.STL" />
+      </geometry>
+    </collision>
+  </link>
+  <gazebo reference="arm_base_link">
         <material>Gazebo/Grey</material>
-        <turnGravityOff>true</turnGravityOff>
-    </gazebo>
-  <joint name="arm_joint" type="fixed">
-			<parent link="${parent}"/>
-			<child link="base_arm_link"/>
-			<origin xyz="${x} ${y} ${z}" rpy="${rx} ${ry} ${rz}" />
-  </joint>
-  <link
-    name="arm_axel">
-    <inertial>
-      <origin
-        xyz="-6.71167554128979E-05 0.147555068632442 -5.01352348164508E-07"
-        rpy="0 0 0" />
-      <mass
-        value="0.116752432749066" />
-      <inertia
-        ixx="0.000715149281043979"
-        ixy="7.80945806556874E-07"
-        ixz="6.95759354868419E-10"
-        iyy="8.63256490972112E-06"
-        iyz="-1.92225108206073E-09"
-        izz="0.000715441962309322" />
-    </inertial>
-    <visual>
-      <origin
-        xyz="0 0 0"
-        rpy="0 0 0" />
-      <geometry>
-        <mesh
-          filename="package://fsr_husky_description/models/arm/arm_axel.STL" />
+	<selfCollide>false</selfCollide>
+        <turnGravityOff>true</turnGravityOff>
+  </gazebo>
+  <link
+    name="arm_axel_link">
+    <inertial>
+      <origin
+        xyz="1.9672E-08 0.14921 0.0024909"
+        rpy="0 0 0" />
+      <mass
+        value="0.14047" />
+      <inertia
+        ixx="0.00082761"
+        ixy="-1.2806E-12"
+        ixz="5.0183E-11"
+        iyy="1.9163E-05"
+        iyz="1.7051E-06"
+        izz="0.00081808" />
+    </inertial>
+    <visual>
+      <origin
+        xyz="0 0 0"
+        rpy="0 0 0" />
+      <geometry>
+        <mesh
+          filename="package://fsr_husky_description/models/arm/arm_axel_link.STL" />
       </geometry>
       <material
@@ -114,22 +110,22 @@
       <geometry>
         <mesh
-          filename="package://fsr_husky_description/models/arm/arm_axel.STL" />
-      </geometry>
-    </collision>
-  </link>
-  <gazebo reference="arm_axel">
+          filename="package://fsr_husky_description/models/arm/arm_axel_link.STL" />
+      </geometry>
+    </collision>
+  </link>
+  <gazebo reference="arm_axel_link">
         <material>Gazebo/Grey</material>
         <turnGravityOff>true</turnGravityOff>
-    </gazebo>
+  </gazebo>
   <joint
     name="arm_axel_joint"
     type="revolute">
     <origin
-      xyz="0.06 0.152 0"
-      rpy="1.5708 0 0" />
+      xyz="-0.26654 -0.21 0.2409"
+      rpy="1.5708 2.7207E-18 0.044449" />
     <parent
-      link="base_arm_link" />
+      link="arm_base_link" />
     <child
-      link="arm_axel" />
+      link="arm_axel_link" />
     <axis
       xyz="0 -1 0" />
@@ -137,30 +133,35 @@
       lower="-1.5708"
       upper="1.5708"
-      effort="100"
-      velocity="0.5" />
-  </joint>
-  <link
-    name="upper_arm">
-    <inertial>
-      <origin
-        xyz="0.000102539584510564 0.025319004836415 0.373317706752181"
-        rpy="0 0 0" />
-      <mass
-        value="0.310661228623748" />
-      <inertia
-        ixx="0.0301188716585458"
-        ixy="-4.68610675580059E-08"
-        ixz="1.48034298202518E-05"
-        iyy="0.0301182394443099"
-        iyz="-0.000152720615635198"
-        izz="8.7451640283179E-05" />
-    </inertial>
-    <visual>
-      <origin
-        xyz="0 0 0"
-        rpy="0 0 0" />
-      <geometry>
-        <mesh
-          filename="package://fsr_husky_description/models/arm/upper_arm.STL" />
+      effort="75"
+      velocity="2" />
+    <!--<safety_controller
+      soft_upper="1.5"
+      soft_lower="-1.5"
+      k_position="1"
+	k_velocity="0" />-->
+  </joint>
+  <link
+    name="upper_arm_link">
+    <inertial>
+      <origin
+        xyz="-0.045308 0.03667 0.27592"
+        rpy="0 0 0" />
+      <mass
+        value="1.2589" />
+      <inertia
+        ixx="0.038361"
+        ixy="2.2286E-05"
+        ixz="0.0034205"
+        iyy="0.040565"
+        iyz="-0.00011324"
+        izz="0.0027942" />
+    </inertial>
+    <visual>
+      <origin
+        xyz="0 0 0"
+        rpy="0 0 0" />
+      <geometry>
+        <mesh
+          filename="package://fsr_husky_description/models/arm/upper_arm_link.STL" />
       </geometry>
       <material
@@ -176,107 +177,107 @@
       <geometry>
         <mesh
-          filename="package://fsr_husky_description/models/arm/upper_arm.STL" />
-      </geometry>
-    </collision>
-  </link>
-  <gazebo reference="upper_arm">
+          filename="package://fsr_husky_description/models/arm/upper_arm_link.STL" />
+      </geometry>
+    </collision>
+  </link>
+  <gazebo reference="upper_arm_link">
         <material>Gazebo/Grey</material>
         <turnGravityOff>true</turnGravityOff>
-    </gazebo>
+  </gazebo>
   <joint
     name="upper_arm_joint"
     type="revolute">
     <origin
-      xyz="0 0.1459 -0.0096445"
-      rpy="-1.5708 0 -1.5708" />
+      xyz="0 0.149 0"
+      rpy="1.5708 -1.2212E-13 -1.5708" />
     <parent
-      link="arm_axel" />
+      link="arm_axel_link" />
     <child
-      link="upper_arm" />
+      link="upper_arm_link" />
     <axis
-      xyz="0 1 0" />
+      xyz="0 -1 0" />
     <limit
-      lower="-0.5"
-      upper="0.25"
-      effort="20"
-      velocity="0.5" />
-  </joint>
-  <link
-    name="metal_detector_arm">
-    <inertial>
-      <origin
-        xyz="0.00200170148149059 -0.0639004587205252 -0.0667324909004516"
-        rpy="0 0 0" />
-      <mass
-	value="0.00001" /><!--value="0.730115545526703" />-->
-      <inertia
-        ixx="0.00564260404067653"
-        ixy="4.21272987506857E-05"
-        ixz="4.78655101148471E-05"
-        iyy="0.00114533989924875"
-        iyz="0.00095063627641457"
-        izz="0.00479397824386875" />
-    </inertial>
-    <visual>
-      <origin
-        xyz="0 0 0"
-        rpy="0 0 0" />
-      <geometry>
-        <mesh
-          filename="package://fsr_husky_description/models/arm/metal_detector_arm.STL" />
+      lower="-0.5236"
+      upper="0.5236"
+      effort="35"
+      velocity="2" />
+  </joint>
+  <link
+    name="metal_detector_arm_link">
+    <inertial>
+      <origin
+        xyz="0.0020016 -0.063902 -0.072539"
+        rpy="0 0 0" />
+      <mass
+        value="0.73012" />
+      <inertia
+        ixx="0.0056833"
+        ixy="4.2128E-05"
+        ixz="4.9113E-05"
+        iyy="0.0011861"
+        iyz="0.00096268"
+        izz="0.0047939" />
+    </inertial>
+    <visual>
+      <origin
+        xyz="0 0 0"
+        rpy="0 0 0" />
+      <geometry>
+        <mesh
+          filename="package://fsr_husky_description/models/arm/metal_detector_arm_link.STL" />
       </geometry>
       <material
         name="DarkGray">
         <color
-          rgba="0.494117647058824 0.494117647058824 0.494117647058824 1" />
-      </material>
-    </visual>
-    <collision>
-      <origin
-        xyz="0 0 0"
-        rpy="0 0 0" />
-      <geometry>
-        <mesh
-          filename="package://fsr_husky_description/models/arm/metal_detector_arm.STL" />
-      </geometry>
-    </collision>
-  </link>
-  <gazebo reference="metal_detector_arm">
+          rgba="0.776470588235294 0.756862745098039 0.737254901960784 1" />
+      </material>
+    </visual>
+    <collision>
+      <origin
+        xyz="0 0 0"
+        rpy="0 0 0" />
+      <geometry>
+        <mesh
+          filename="package://fsr_husky_description/models/arm/metal_detector_arm_link.STL" />
+      </geometry>
+    </collision>
+  </link>
+  <gazebo reference="metal_detector_arm_link">
         <material>Gazebo/Grey</material>
         <turnGravityOff>true</turnGravityOff>
-    </gazebo>
+  </gazebo>
   <joint
     name="metal_detector_arm_joint"
     type="revolute">
+    <origin
+      xyz="0 0.0062947 0.8475"
+      rpy="1.5708 -1.5708 0" />
+    <parent
+      link="upper_arm_link" />
+    <child
+      link="metal_detector_arm_link" />
+    <axis
+      xyz="0 0 1" />
+    <limit
+      lower="-0.5236"
+      upper="0.5236"
+      effort="35"
+      velocity="2" />
     <mimic
       joint="upper_arm_joint"
       multiplier="-1" />
-    <origin
-      xyz="0 0 0.8475"
-      rpy="1.5708 -1.5708 0" />
-    <parent
-      link="upper_arm" />
-    <child
-      link="metal_detector_arm" />
-    <axis
-      xyz="0 0 -1" />
-    <limit
-      lower="-0.25"
-      upper="0.5"
-      effort="20"
-      velocity="0.5" />
-  </joint>
-  <link
-    name="metal_detector_antenna">
-    <inertial>
-      <origin
-        xyz="3.6833E-07 0.011468 -0.12477"
-        rpy="0 0 0" />
-      <mass
-	value="12.099" />
+  </joint>
+  <link
+    name="metal_detector_antenna_link">
+    <inertial>
+      <origin
+        xyz="3.7915E-07 0.011468 -0.12477"
+        rpy="0 0 0" />
+      <mass
+        value="12.099" />
       <inertia
         ixx="0.060468"
-        ixy="-4.3221E-09"
-        ixz="5.3405E-07"
+        ixy="-4.2864E-09"
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
File: fsr_husky_description/urdf/fsr_husky_mine_detection.urdf.xacro (robot description, xacro)
@@ -181,5 +181,5 @@
     <!-- FSR Husky Stuff -->
     <!-- BRIDGE macros -->
-    <husky_bridge prefix="front" parent="base_link" x="0.17" y="0" z="${base_z_size}" rx="0" ry="0" rz="0" />
+    <husky_bridge prefix="front" parent="base_link" x="0.09" y="0" z="${base_z_size}" rx="0" ry="0" rz="0" />
     <husky_bridge prefix="back" parent="base_link" x="-0.18" y="0" z="${base_z_size}" rx="0" ry="0" rz="0" />
     <!-- MTi macro -->
@@ -197,5 +197,5 @@
     <alfa_tube2h parent="back_husky_bridge" x="0" y="-0.17" z="0" rx="0" ry="0" rz="0" />
     <!-- FSR Husky De-mining Arm -->
-    <fsr_husky_arm parent="base_link" x="0.120" y="-0.15" z="${base_z_size}" rx="0" ry="0" rz="0" />
+    <fsr_husky_arm parent="base_link" x="-0.025" y="-0.21" z="0.007" rx="0" ry="0" rz="3.14" />
     <gazebo>
       <plugin name="gazebo_ros_control" filename="libgazebo_ros_control.so">

Commit message: Update to the metal detector arm length on the URDF model.

File: fsr_husky_description/urdf/arm/fsr_husky_arm.urdf.xacro (robot description, xacro)
@@ -78,5 +78,5 @@
     <inertial>
       <origin
-        xyz="1.9672E-08 0.14921 0.0024909"
+        xyz="1.8559E-08 0.14921 0.0024909"
         rpy="0 0 0" />
       <mass
@@ -84,6 +84,6 @@
       <inertia
         ixx="0.00082761"
-        ixy="-1.2806E-12"
-        ixz="5.0183E-11"
+        ixy="1.0013E-11"
+        ixz="4.7857E-11"
         iyy="1.9163E-05"
         iyz="1.7051E-06"
@@ -123,5 +123,5 @@
     <origin
       xyz="-0.26654 -0.21 0.2409"
-      rpy="1.5708 2.7207E-18 0.044449" />
+      rpy="1.5708 0 0" />
     <parent
       link="arm_base_link" />
@@ -145,15 +145,15 @@
     <inertial>
       <origin
-        xyz="-0.045308 0.03667 0.27592"
+        xyz="-0.050412 0.036759 0.30862"
         rpy="0 0 0" />
       <mass
-        value="1.2589" />
+        value="1.3043" />
       <inertia
-        ixx="0.038361"
-        ixy="2.2286E-05"
-        ixz="0.0034205"
-        iyy="0.040565"
-        iyz="-0.00011324"
-        izz="0.0027942" />
+      ixx="0.067422"
+      ixy="1.8427E-05"
+      ixz="0.0058821"
+      iyy="0.070529"
+      iyz="-0.00013128"
+      izz="0.0037085" />
     </inertial>
     <visual>
@@ -190,5 +190,5 @@
     <origin
       xyz="0 0.149 0"
-      rpy="1.5708 -1.2212E-13 -1.5708" />
+      rpy="1.5708 0 -1.5708" />
     <parent
       link="arm_axel_link" />
@@ -206,15 +206,15 @@
     name="metal_detector_arm_link">
     <inertial>
-      <origin
-        xyz="0.0020016 -0.063902 -0.072539"
-        rpy="0 0 0" />
-      <mass
+        <origin
+        xyz="-0.0020016 0.063902 -0.069765"
+        rpy="0 0 0" />
+        <mass
         value="0.73012" />
-      <inertia
+        <inertia
         ixx="0.0056833"
         ixy="4.2128E-05"
-        ixz="4.9113E-05"
+        ixz="-4.9113E-05"
         iyy="0.0011861"
-        iyz="0.00096268"
+        iyz="-0.00096268"
         izz="0.0047939" />
     </inertial>
@@ -251,6 +251,6 @@
     type="revolute">
     <origin
-      xyz="0 0.0062947 0.8475"
-      rpy="1.5708 -1.5708 0" />
+    xyz="0 0.0090687 1.0475"
+    rpy="1.5708 1.5708 0" />
     <parent
       link="upper_arm_link" />
@@ -276,8 +276,8 @@
       <mass
         value="12.099" />
-      <inertia
+        <inertia
         ixx="0.060468"
-        ixy="-4.2864E-09"
-        ixz="5.461E-07"
+        ixy="-4.3221E-09"
+        ixz="5.3405E-07"
         iyy="0.27654"
         iyz="-0.0010461"
@@ -316,6 +316,6 @@
     type="fixed">
     <origin
-      xyz="0 -0.33276 0.090995"
-      rpy="2.7728E-15 2.7756E-15 1.2333E-16" />
+    xyz="0 0.33276 0.093769"
+    rpy="0 0 3.1416" />
     <parent
       link="metal_detector_arm_link" />
@@ -328,16 +328,16 @@
     name="lower_arm_link">
     <inertial>
-      <origin
-        xyz="-3.74E-08 0.061694 0.38021"
-        rpy="0 0 0" />
-      <mass
-        value="0.31529" />
-      <inertia
-        ixx="0.031123"
-        ixy="-2.3256E-10"
-        ixz="3.6524E-09"
-        iyy="0.031122"
-        iyz="-0.00015585"
-        izz="8.7836E-05" />
+        <origin
+        xyz="-3.5256E-08 0.024129 0.47631"
+        rpy="0 0 0" />
+        <mass
+        value="0.36063" />
+        <inertia
+        ixx="0.05231"
+        ixy="-2.4697E-10"
+        ixz="5.203E-09"
+        iyy="0.05231"
+        iyz="-0.00019955"
+        izz="0.00010017" />
     </inertial>
     <visual>
@@ -373,6 +373,6 @@
     type="revolute">
     <origin
-      xyz="0 0.084 -0.023752"
-      rpy="1.5708 -1.2212E-13 -1.5708" />
+    xyz="0 0.084 0.013631"
+    rpy="1.5708 0 -1.5708" />
     <parent
       link="arm_axel_link" />
